File: Mothbox_PCBs/Mothbox_PCB_5.0.6/MothBox/GPS.kicad_sch (KiCad schematic)
At the start: 22 parts, among them J5 Conn_1.25mm, Q13 AP30P30Q, U10 Days, U11 Hours3, U12 MODE, U13 Hours1, U14 Hours2, U15 PCA9555PW, U16 PCA9555PW, U17 DS18B20U, U18 LTR-303ALS-01, U8 GPs 5 pin PM2.54-1*5, U9 PCA9555PW

Commit message: Passes Stricter DRC. Shifted Temp sensor. Rotated switches correctly
Parts:
- U10: value Days -> hours_3
- U11: value Hours3 -> Days
Connections:
- net Armed/Disarmed: now also U11.8; no longer U11.16
- net Attractor_1: now also U12.5; no longer U12.13
- net Attractor_2: now also U12.4; no longer U12.12
- net Attractor_3: now also U12.3; no longer U12.11
- net C1: now also U12.2; no longer U12.10
- net C2: now also U12.1; no longer U12.9
- net Fri: now also U11.5; no longer U11.13
- net GND: now also U10.10, U10.11, U10.12, U10.13, U10.14, U10.15, U10.16, U10.9, U11.10, U11.11, U11.12, U11.13, U11.14, U11.15, U11.16, U11.9, U12.10, U12.11, U12.12, U12.13, U12.14, U12.15, U12.16, U12.9, U13.10, U13.11, U13.12, U13.13, U13.14, U13.15, U13.16, U13.9, U14.10, U14.11, U14.12, U14.13, U14.14, U14.15, U14.16, U14.9; no longer U10.1, U10.2, U10.3, U10.4, U10.5, U10.6, U10.7, U10.8, U11.1, U11.2, U11.3, U11.4, U11.5, U11.6, U11.7, U11.8, U12.1, U12.2, U12.3, U12.4, U12.5, U12.6, U12.7, U12.8, U13.1, U13.2, U13.3, U13.4, U13.5, U13.6, U13.7, U13.8, U14.1, U14.2, U14.3, U14.4, U14.5, U14.6, U14.7, U14.8
- net HI/LOW_PWR: now also U12.7; no longer U12.15
- net Hour_1: now also U13.8; no longer U13.16
- net Hour_10: now also U14.7; no longer U14.15
- net Hour_11: now also U14.6; no longer U14.14
- net Hour_12: now also U14.5; no longer U14.13
- net Hour_13: now also U14.4; no longer U14.12
- net Hour_14: now also U14.3; no longer U14.11
- net Hour_15: now also U14.2; no longer U14.10
- net Hour_16: now also U14.1; no longer U14.9
- net Hour_17: now also U10.7; no longer U10.15
- net Hour_18: now also U10.6; no longer U10.14
- net Hour_19: now also U10.5; no longer U10.13
- net Hour_2: now also U13.7; no longer U13.15
- net Hour_20: now also U10.4; no longer U10.12
- net Hour_21: now also U10.3; no longer U10.11
- net Hour_22: now also U10.2; no longer U10.10
- net Hour_23: now also U10.1; no longer U10.9
- net Hour_24: now also U10.8; no longer U10.16
- net Hour_3: now also U13.6; no longer U13.14
- net Hour_4: now also U13.5; no longer U13.13
- net Hour_5: now also U13.4; no longer U13.12
- net Hour_6: now also U13.3; no longer U13.11
- net Hour_7: now also U13.2; no longer U13.10
- net Hour_8: now also U13.1; no longer U13.9
- net Hour_9: now also U14.8; no longer U14.16
- net INT/EXT_Attractor: now also U12.6; no longer U12.14
- net Mon: now also U11.1; no longer U11.9
- net Sat: now also U11.6; no longer U11.14
- net Sun: now also U11.7; no longer U11.15
- net Test_Debug: now also U12.8; no longer U12.16
- net Thur: now also U11.4; no longer U11.12
- net Tue: now also U11.2; no longer U11.10
- net Wed: now also U11.3; no longer U11.11
