File: Mothbox_PCBs/Mothbox_PCB_5.0.6/MothBox/Mothbox_5.0.6.kicad_pcb (KiCad board)
At the start: 2 copper layers, 237 x 139 mm, 182 parts, among them J1 DB141V-2.54-4P, J2 DB141V-2.54-4P, J3 DB141V-2.54-4P, J4 DB141V-2.54-4P, J5 Conn_1.25mm, Q1 AP30P30Q, Q10 AP30P30Q, Q13 AP30P30Q, Q2 AO3400A, Q3 YJQ10N2A, Q4 YJQ10N2A, Q5 YJQ10N2A, Q6 YJQ10N2A, Q7 YJQ10N2A, Q8 AP30P30Q, Q9 YJQ10N2A, SW2 4-1437565-1, U10 Days, U11 Hours3, U12 MODE, U13 Hours1, U14 Hours2, U15 PCA9555PW, U16 PCA9555PW, U17 DS18B20U, U18 LTR-303ALS-01, U19 graphic, U2 XL4015E1, U3 TI INA219AIDCNR, U5 RASPBERRY_PI_5, U6 RASPBERRY_PI_4B_4GB, U7 Female Inv Socket Pi 2.54-2*20, U8 GPs 5 pin PM2.54-1*5, U9 PCA9555PW

Commit message: Added Holes for Attractor, Added Holes for corners instead of screws, widened pi hole
Parts:
- added ?: , , F.Cu at (49.5, 23.8)
- added ?: , , F.Cu at (199.0, 21.3)
- added ?: , , F.Cu at (142.0, 21.8)
- moved LED43 10.5 mm to (109.0, 138.8)
- moved LED44 10.4 mm to (108.0, 121.3)
- moved LED5 7.68 mm to (122.5, 100.3)
- moved TP6 6.47 mm to (239.5, 73.3)
- moved R18 4.64 mm to (122.5, 88.3)
- moved LED18 4.23 mm to (45.0, 104.8), turned to -90 degrees
- moved LED4 1.77 mm to (124.5, 72.3)
- moved LED45 1.05 mm to (122.5, 119.0)
Routing:
- net Net-(LED12-K): track 453.7 -> 444.3 mm
- net Net-(LED4-K): track 28.3 -> 37.1 mm
- net Net-(LED5-K): track 23.3 -> 31.2 mm
- net Net-(LED44-K): track 8.62 -> 15.0 mm
- net Net-(LED27-K): track 481.2 -> 487.5 mm
- net Net-(LED43-K): track 15.5 -> 20.1 mm
- net +12V: track 797.9 -> 802.1 mm
- net Net-(LED17-K): track 9.14 -> 6.66 mm
- net Net-(LED4-A): track 17.8 -> 16.5 mm
- net UV3_CTRL: track 136.6 -> 137.3 mm
- net Net-(LED43-A): track 30.0 -> 29.5 mm
- net GND: vias 927 -> 926
Other:
- outline, holes or cut-outs redrawn
- board text added: "V5.0.6"
- board text removed: "V5.0.5"

Commit message: Passes Stricter DRC. Shifted Temp sensor. Rotated switches correctly
Parts:
- R32: value 0R -> (actually 0R now not 100R)
- SW2: value 4-1437565-1 -> KH-6X6X5H-STM
- U10: value Days -> hours_3
- U11: value Hours3 -> Days
- U3: value TI INA219AIDCNR -> INA219BIDCNT; footprint easyeda2kicad:SOT-23-8_L3.0-W1.7-P0.65-LS2.8-BR -> MothBox_footprints_Library:SOT-23-8
- moved C10 6.82 mm to (241.2, 90.5)
- moved C11 6.82 mm to (239.5, 90.5)
- moved C4 5.79 mm to (220.5, 90.2)
- moved R33 5.79 mm to (216.1, 92.7)
- moved U17 5.79 mm to (216.2, 90.1)
- moved C16 5.32 mm to (229.0, 86.7)
- moved J5 5.26 mm to (216.5, 82.8)
- moved U10 0.34 mm to (182.3, 27.4), turned to 180 degrees
- moved U14 0.32 mm to (217.2, 27.2), turned to 180 degrees
- moved H4 0.28 mm to (41.3, 28.0)
- moved U13 0.11 mm to (238.7, 27.0), turned to 180 degrees
- moved U12 0.06 mm to (149.5, 46.8), turned to 180 degrees
- turned U11 to 180 degrees
- turned U3 to 0 degrees
Connections:
- U10 pad 1: GND -> /GPS and Switches and Light Sensor/Hour_23
- U10 pad 10: /GPS and Switches and Light Sensor/Hour_22 -> GND
- U10 pad 11: /GPS and Switches and Light Sensor/Hour_21 -> GND
- U10 pad 12: /GPS and Switches and Light Sensor/Hour_20 -> GND
- U10 pad 13: /GPS and Switches and Light Sensor/Hour_19 -> GND
- U10 pad 14: /GPS and Switches and Light Sensor/Hour_18 -> GND
- U10 pad 15: /GPS and Switches and Light Sensor/Hour_17 -> GND
- U10 pad 16: /GPS and Switches and Light Sensor/Hour_24 -> GND
- U10 pad 2: GND -> /GPS and Switches and Light Sensor/Hour_22
- U10 pad 3: GND -> /GPS and Switches and Light Sensor/Hour_21
- U10 pad 4: GND -> /GPS and Switches and Light Sensor/Hour_20
- U10 pad 5: GND -> /GPS and Switches and Light Sensor/Hour_19
- U10 pad 6: GND -> /GPS and Switches and Light Sensor/Hour_18
- U10 pad 7: GND -> /GPS and Switches and Light Sensor/Hour_17
- U10 pad 8: GND -> /GPS and Switches and Light Sensor/Hour_24
- U10 pad 9: /GPS and Switches and Light Sensor/Hour_23 -> GND
- U11 pad 1: GND -> /GPS and Switches and Light Sensor/Mon
- U11 pad 10: /GPS and Switches and Light Sensor/Tue -> GND
- U11 pad 11: /GPS and Switches and Light Sensor/Wed -> GND
- U11 pad 12: /GPS and Switches and Light Sensor/Thur -> GND
- U11 pad 13: /GPS and Switches and Light Sensor/Fri -> GND
- U11 pad 14: /GPS and Switches and Light Sensor/Sat -> GND
- U11 pad 15: /GPS and Switches and Light Sensor/Sun -> GND
- U11 pad 16: /GPS and Switches and Light Sensor/Armed/Disarmed -> GND
- U11 pad 2: GND -> /GPS and Switches and Light Sensor/Tue
- U11 pad 3: GND -> /GPS and Switches and Light Sensor/Wed
- U11 pad 4: GND -> /GPS and Switches and Light Sensor/Thur
- U11 pad 5: GND -> /GPS and Switches and Light Sensor/Fri
- U11 pad 6: GND -> /GPS and Switches and Light Sensor/Sat
- U11 pad 7: GND -> /GPS and Switches and Light Sensor/Sun
- U11 pad 8: GND -> /GPS and Switches and Light Sensor/Armed/Disarmed
- U11 pad 9: /GPS and Switches and Light Sensor/Mon -> GND
- U12 pad 1: GND -> /GPS and Switches and Light Sensor/C2
- U12 pad 10: /GPS and Switches and Light Sensor/C1 -> GND
- U12 pad 11: /GPS and Switches and Light Sensor/Attractor_3 -> GND
- U12 pad 12: /GPS and Switches and Light Sensor/Attractor_2 -> GND
- U12 pad 13: /GPS and Switches and Light Sensor/Attractor_1 -> GND
- U12 pad 14: /GPS and Switches and Light Sensor/INT/EXT_Attractor -> GND
- U12 pad 15: /GPS and Switches and Light Sensor/HI/LOW_PWR -> GND
- U12 pad 16: /GPS and Switches and Light Sensor/Test_Debug -> GND
- U12 pad 2: GND -> /GPS and Switches and Light Sensor/C1
- U12 pad 3: GND -> /GPS and Switches and Light Sensor/Attractor_3
- U12 pad 4: GND -> /GPS and Switches and Light Sensor/Attractor_2
- U12 pad 5: GND -> /GPS and Switches and Light Sensor/Attractor_1
- U12 pad 6: GND -> /GPS and Switches and Light Sensor/INT/EXT_Attractor
- U12 pad 7: GND -> /GPS and Switches and Light Sensor/HI/LOW_PWR
- U12 pad 8: GND -> /GPS and Switches and Light Sensor/Test_Debug
- U12 pad 9: /GPS and Switches and Light Sensor/C2 -> GND
- U13 pad 1: GND -> /GPS and Switches and Light Sensor/Hour_8
- U13 pad 10: /GPS and Switches and Light Sensor/Hour_7 -> GND
- U13 pad 11: /GPS and Switches and Light Sensor/Hour_6 -> GND
- U13 pad 12: /GPS and Switches and Light Sensor/Hour_5 -> GND
- U13 pad 13: /GPS and Switches and Light Sensor/Hour_4 -> GND
- U13 pad 14: /GPS and Switches and Light Sensor/Hour_3 -> GND
- U13 pad 15: /GPS and Switches and Light Sensor/Hour_2 -> GND
- U13 pad 16: /GPS and Switches and Light Sensor/Hour_1 -> GND
- U13 pad 2: GND -> /GPS and Switches and Light Sensor/Hour_7
- U13 pad 3: GND -> /GPS and Switches and Light Sensor/Hour_6
- U13 pad 4: GND -> /GPS and Switches and Light Sensor/Hour_5
- U13 pad 5: GND -> /GPS and Switches and Light Sensor/Hour_4
- U13 pad 6: GND -> /GPS and Switches and Light Sensor/Hour_3
- U13 pad 7: GND -> /GPS and Switches and Light Sensor/Hour_2
- U13 pad 8: GND -> /GPS and Switches and Light Sensor/Hour_1
- U13 pad 9: /GPS and Switches and Light Sensor/Hour_8 -> GND
- U14 pad 1: GND -> /GPS and Switches and Light Sensor/Hour_16
- U14 pad 10: /GPS and Switches and Light Sensor/Hour_15 -> GND
- U14 pad 11: /GPS and Switches and Light Sensor/Hour_14 -> GND
- U14 pad 12: /GPS and Switches and Light Sensor/Hour_13 -> GND
- U14 pad 13: /GPS and Switches and Light Sensor/Hour_12 -> GND
- U14 pad 14: /GPS and Switches and Light Sensor/Hour_11 -> GND
- U14 pad 15: /GPS and Switches and Light Sensor/Hour_10 -> GND
- U14 pad 16: /GPS and Switches and Light Sensor/Hour_9 -> GND
- U14 pad 2: GND -> /GPS and Switches and Light Sensor/Hour_15
- U14 pad 3: GND -> /GPS and Switches and Light Sensor/Hour_14
- U14 pad 4: GND -> /GPS and Switches and Light Sensor/Hour_13
- U14 pad 5: GND -> /GPS and Switches and Light Sensor/Hour_12
- U14 pad 6: GND -> /GPS and Switches and Light Sensor/Hour_11
- U14 pad 7: GND -> /GPS and Switches and Light Sensor/Hour_10
- U14 pad 8: GND -> /GPS and Switches and Light Sensor/Hour_9
- U14 pad 9: /GPS and Switches and Light Sensor/Hour_16 -> GND
Routing:
- net +5V: track 455.9 -> 497.9 mm, vias 5 -> 9
- net +12V: track 802.1 -> 811.3 mm
- net +3.3V: track 444.5 -> 450.4 mm
- net GPIO4: track 184.3 -> 189.6 mm
- net GND: track 437.4 -> 442.3 mm, vias 926 -> 936
- net Net-(J4-Pin_1): track 28.0 -> 31.6 mm
- net SCL: track 372.6 -> 374.1 mm
- net Net-(LED12-K): track 444.3 -> 443.5 mm
- net GPS_RX: track 185.0 -> 185.7 mm
- net GPS_PPS: track 147.7 -> 148.3 mm
Other:
- outline, holes or cut-outs redrawn
- board text added: "MOTHBOX V5.0.6"
- board text removed: "MOTHBOX V5.0.5"
