File: Mothbox_PCBs/Mothbox_PCB_5.0.6/MothBox/Mothbox_5.0.6.kicad_pcb (KiCad board)
At the start: 2 copper layers, 237 x 139.1 mm, 185 parts, among them J1 DB141V-2.54-4P, J2 DB141V-2.54-4P, J3 DB141V-2.54-4P, J4 DB141V-2.54-4P, J5 Conn_1.25mm, Q1 AP30P30Q, Q10 AP30P30Q, Q13 AP30P30Q, Q2 AO3400A, Q3 YJQ10N2A, Q4 YJQ10N2A, Q5 YJQ10N2A, Q6 YJQ10N2A, Q7 YJQ10N2A, Q8 AP30P30Q, Q9 YJQ10N2A, SW2 KH-6X6X5H-STM, U10 hours_3, U11 Days, U12 MODE, U13 Hours1, U14 Hours2, U15 PCA9555PW, U16 PCA9555PW, U17 DS18B20U, U18 LITEON LTR-F216A, U19 graphic, U2 XL4015E1, U3 INA219BIDCNT, U5 RASPBERRY_PI_5, U6 RASPBERRY_PI_4B_4GB, U7 Female Inv Socket Pi 2.54-2*20, U8 GPs 5 pin PM2.54-1*5, U9 PCA9555PW

Commit message: added missing c14 c16 capacitors in
Parts:
- C14, C16: footprint easyeda2kicad:CAP-SMD_BD12.5-L13.0-W13.0-RD -> EasyEDA:CAP-SMD_BD12.5-L13.0-W13.0-RD
Changed lines of the file:
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@@
 		)
 	)
-	(footprint "easyeda2kicad:CAP-SMD_BD12.5-L13.0-W13.0-RD"
+	(footprint "EasyEDA:CAP-SMD_BD12.5-L13.0-W13.0-RD"
 		(layer "B.Cu")
 		(at 229 86.701703 -90)
+		(descr "470uF 50V ±20%")
 		(property "Reference" "C16"
 			(at 0 4 90)
@@
 				(font
 					(size 1.27 1.27)
-					(thickness 0.15)
 				)
 				(justify mirror)
@@
 				(font
 					(size 1.27 1.27)
-					(thickness 0.15)
+				)
+				(justify mirror)
+			)
+		)
+		(property "LCSC Part" "C90272"
+			(at 0 0 90)
+			(layer "B.Fab")
+			(hide yes)
+			(effects
+				(font
+					(size 1.27 1.27)
 				)
 				(justify mirror)
@@
 			)
 		)
-		(property "LCSC_Part" "C90272"
-			(at 0 0 270)
-			(unlocked yes)
-			(layer "B.Fab")
-			(hide yes)
-			(effects
-				(font
-					(size 1 1)
-					(thickness 0.15)
-				)
-				(justify mirror)
-			)
-		)
 		(property ki_fp_filters "CP_*")
 		(sheetname "/Power/")
 		(sheetfile "Power.kicad_sch")
-		(units
-			(unit
-				(name "A")
-				(pins "1" "2")
-			)
-		)
-		(attr smd dnp)
+		(attr smd)
 		(duplicate_pad_numbers_are_jumpers no)
 		(fp_line
@@
 		)
 		(fp_arc
-			(start 6.0602 1.088957)
-			(mid 0.051521 6.09981)
+			(start 6.062414 1.07732)
+			(mid 0.057444 6.099757)
 			(end -6.04 1.19)
 			(stroke
@@
 		)
 		(fp_arc
-			(start -6.007911 -1.271112)
-			(mid 0.087846 -6.013191)
+			(start -6.004745 -1.287299)
+			(mid 0.096091 -6.029095)
 			(end 6.03 -1.08)
 			(stroke
@@
 			)
 			(fill no)
-			(layer "B.Fab")
+			(layer "B.SilkS")
+		)
+		(fp_poly
+			(pts
+				(xy -1.569999 -5.919978) (xy -1.589989 5.969991) (xy -2.250008 5.719978) (xy -2.910002 5.489981)
+				(xy -3.419983 5.159985) (xy -3.750005 4.88) (xy -4.239997 4.549978) (xy -4.619981 4.139997) (xy -5.069992 3.559988)
+				(xy -5.299989 3.019984) (xy -5.579999 2.619985) (xy -5.709996 2.159991) (xy -5.889981 1.740002)
+				(xy -5.999988 1.419987) (xy -6.039993 1.159993) (xy -6.039993 1.110005) (xy -2.949956 1.119886)
+				(xy -2.950007 -0.049987) (xy -2.949956 -1.229868) (xy -5.999988 -1.249985) (xy -5.850001 -1.829994)
+				(xy -5.639994 -2.449982) (xy -5.289982 -3.129991) (xy -4.950003 -3.699993) (xy -4.569993 -4.119982)
+				(xy -4.269994 -4.449978) (xy -3.839997 -4.81998) (xy -3.159989 -5.249977) (xy -2.149983 -5.749976)
+				(xy -1.580007 -5.950001) (xy -1.569999 -5.919978)
+			)
+			(stroke
+				(width 0)
+				(type solid)
+			)
+			(fill yes)
+			(layer "B.SilkS")
+		)
+		(fp_line
+			(start -6.5 6.5)
+			(end 3.5 6.5)
+			(stroke
+				(width 0.05)
+				(type solid)
+			)
+			(layer "B.CrtYd")
+		)
+		(fp_line
+			(start 3.5 6.5)
+			(end 6.5 3.5)
+			(stroke
+				(width 0.05)
+				(type solid)
+			)
+			(layer "B.CrtYd")
+		)
+		(fp_line
+			(start 6.5 3.5)
+			(end 6.5 -3.5)
+			(stroke
+				(width 0.05)
+				(type solid)
+			)
+			(layer "B.CrtYd")
+		)
+		(fp_line
+			(start 6.5 -3.5)
+			(end 3.5 -6.5)
+			(stroke
+				(width 0.05)
+				(type solid)
+			)
+			(layer "B.CrtYd")
+		)
+		(fp_line
+			(start -6.5 -6.5)
+			(end -6.5 6.5)
+			(stroke
+				(width 0.05)
+				(type solid)
+			)
+			(layer "B.CrtYd")
+		)
+		(fp_line
+			(start 3.5 -6.5)
+			(end -6.5 -6.5)
+			(stroke
+				(width 0.05)
+				(type solid)
+			)
+			(layer "B.CrtYd")
 		)
 		(fp_text user "${REFERENCE}"
@@
 		)
 		(embedded_fonts no)
-		(model "${EASYEDA2KICAD}/easyeda2kicad.3dshapes/CAP-SMD_D12.5-L13.0-W13.0-H13.5.wrl"
+		(model "${KIPRJMOD}/EasyEDA.3dshapes/CAP-SMD_D12.5-L13.0-W13.0-H13.5.wrl"
 			(offset
-				(xyz 0 -0 -0)
+				(xyz 0 0 0)
 			)
 			(scale
@@
 		)
 	)
-	(footprint "easyeda2kicad:CAP-SMD_BD12.5-L13.0-W13.0-RD"
+	(footprint "EasyEDA:CAP-SMD_BD12.5-L13.0-W13.0-RD"
 		(layer "B.Cu")
 		(at 231.884092 127.527159)
+		(descr "470uF 50V ±20%")
 		(property "Reference" "C14"
 			(at 0 4 180)
@@
 				(font
 					(size 1.27 1.27)
-					(thickness 0.15)
 				)
 				(justify mirror)
@@
 				(font
 					(size 1.27 1.27)
-					(thickness 0.15)
+				)
+				(justify mirror)
+			)
+		)
+		(property "LCSC Part" "C90272"
+			(at 0 0 180)
+			(layer "B.Fab")
+			(hide yes)
+			(effects
+				(font
+					(size 1.27 1.27)
 				)
 				(justify mirror)
@@
 			)
 		)
-		(property "LCSC_Part" "C90272"
-			(at 0 0 180)
-			(unlocked yes)
-			(layer "B.Fab")
-			(hide yes)
-			(effects
-				(font
-					(size 1 1)
-					(thickness 0.15)
-				)
-				(justify mirror)
-			)
-		)
 		(property ki_fp_filters "CP_*")
 		(sheetname "/Power/")
 		(sheetfile "Power.kicad_sch")
-		(units
-			(unit
-				(name "A")
-				(pins "1" "2")
-			)
-		)
-		(attr smd dnp)
+		(attr smd)
 		(duplicate_pad_numbers_are_jumpers no)
 		(fp_line
@@
 		)
 		(fp_arc
-			(start -6.007911 -1.271112)
-			(mid 0.087846 -6.013191)
+			(start -6.004745 -1.287299)
+			(mid 0.096091 -6.029095)
 			(end 6.03 -1.08)
 			(stroke
@@
 		)
 		(fp_arc
-			(start 6.0602 1.088957)
-			(mid 0.051521 6.09981)
+			(start 6.062414 1.07732)
+			(mid 0.057444 6.099757)
 			(end -6.04 1.19)
 			(stroke
@@
 			)
 			(fill no)
-			(layer "B.Fab")
+			(layer "B.SilkS")
+		)
+		(fp_poly
+			(pts
+				(xy -1.569999 -5.919978) (xy -1.589989 5.969991) (xy -2.250008 5.719978) (xy -2.910002 5.489981)
+				(xy -3.419983 5.159985) (xy -3.750005 4.88) (xy -4.239997 4.549978) (xy -4.619981 4.139997) (xy -5.069992 3.559988)
+				(xy -5.299989 3.019984) (xy -5.579999 2.619985) (xy -5.709996 2.159991) (xy -5.889981 1.740002)
+				(xy -5.999988 1.419987) (xy -6.039993 1.159993) (xy -6.039993 1.110005) (xy -2.949956 1.119886)
+				(xy -2.950007 -0.049987) (xy -2.949956 -1.229868) (xy -5.999988 -1.249985) (xy -5.850001 -1.829994)
+				(xy -5.639994 -2.449982) (xy -5.289982 -3.129991) (xy -4.950003 -3.699993) (xy -4.569993 -4.119982)
+				(xy -4.269994 -4.449978) (xy -3.839997 -4.81998) (xy -3.159989 -5.249977) (xy -2.149983 -5.749976)
+				(xy -1.580007 -5.950001) (xy -1.569999 -5.919978)
+			)
+			(stroke
+				(width 0)
+				(type solid)
+			)
+			(fill yes)
+			(layer "B.SilkS")
+		)
+		(fp_line
+			(start -6.5 -6.5)
+			(end -6.5 6.5)
+			(stroke
+				(width 0.05)
+				(type solid)
+			)
+			(layer "B.CrtYd")
+		)
+		(fp_line
+			(start -6.5 6.5)
+			(end 3.5 6.5)
+			(stroke
+				(width 0.05)
+				(type solid)
+			)
+			(layer "B.CrtYd")
+		)
+		(fp_line
+			(start 3.5 -6.5)
+			(end -6.5 -6.5)
+			(stroke
+				(width 0.05)
+				(type solid)
+			)
+			(layer "B.CrtYd")
+		)
+		(fp_line
+			(start 3.5 6.5)
+			(end 6.5 3.5)
+			(stroke
+				(width 0.05)
+				(type solid)
+			)
+			(layer "B.CrtYd")
+		)
+		(fp_line
+			(start 6.5 -3.5)
+			(end 3.5 -6.5)
+			(stroke
+				(width 0.05)
+				(type solid)
+			)
+			(layer "B.CrtYd")
+		)
+		(fp_line
+			(start 6.5 3.5)
+			(end 6.5 -3.5)
+			(stroke
+				(width 0.05)
+				(type solid)
+			)
+			(layer "B.CrtYd")
 		)
 		(fp_text user "${REFERENCE}"
@@
 		)
 		(embedded_fonts no)
-		(model "${EASYEDA2KICAD}/easyeda2kicad.3dshapes/CAP-SMD_D12.5-L13.0-W13.0-H13.5.wrl"
+		(model "${KIPRJMOD}/EasyEDA.3dshapes/CAP-SMD_D12.5-L13.0-W13.0-H13.5.wrl"
 			(offset
-				(xyz 0 -0 -0)
+				(xyz 0 0 0)
 			)
 			(scale
