File: Mothbox_PCBs/Mothbox_PCB_5.0.6/MothBox/Power.kicad_sch (KiCad schematic)
At the start: 50 parts, among them J1 DB141V-2.54-4P, J2 DB141V-2.54-4P, J3 DB141V-2.54-4P, Q1 AP30P30Q, Q10 AP30P30Q, Q2 AO3400A, Q8 AP30P30Q, SW2 KH-6X6X5H-STM, U1 Place Holder voltage regulator, U2 XL4015E1, U3 INA219BIDCNT

Commit message: Passes Stricter DRC. Shifted Temp sensor. Rotated switches correctly
Parts:
- D1, D2, D4: DESCRIPTION MM1W18 -> (none)
