File: Mothbeam_PCBs/AndyMothbeam_forMBv5.0.3/Mothbeam_Visible_450_520_White/Mothbeam.kicad_pcb (KiCad board)
At the start: 2 copper layers, 27.8 x 45 mm, 24 parts, among them CN1 X6511FRS-04-C85D30, SW2 SW_DIP_x04, U1 BCR421U, U2 BCR421U, U3 BCR421U

Commit message: Starting to add holes back to mothbeams!
Parts:
- added ?: , , F.Cu at (124.0, 32.4)
- added REF**: MountingHole_3.2mm_M3, MountingHole:MountingHole_3.2mm_M3, F.Cu at (102.2, 32.8)
